File: PCB/WLED_Box.kicad_pcb (KiCad board)
At the start: 2 copper layers, 23 x 50.5 mm, 7 parts, among them J1 USB_C_Receptacle_PowerOnly_6P, J2 Conn_01x03_Socket, U1 XIAO-ESP32-C3-DIP

Commit message: CAD Finishing
Other:
- board text added: "Data"
- board text added: "GND"
- board text added: "VCC"
Changed lines of the file:
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@@
+		)
+	)
+	(gr_text "Data"
+		(at 129 57.77 270)
+		(layer "F.SilkS")
+		(effects
+			(font
+				(size 1 1)
+				(thickness 0.1)
+			)
+			(justify left bottom)
+		)
+	)
+	(gr_text "GND\n"
+		(at 134 57 0)
+		(layer "F.SilkS")
+		(effects
+			(font
+				(size 1 1)
+				(thickness 0.1)
+			)
+			(justify left bottom)
+		)
+	)
+	(gr_text "VCC\n"
+		(at 122 57 0)
+		(layer "F.SilkS")
+		(effects
+			(font
+				(size 1 1)
+				(thickness 0.1)
+			)
+			(justify left bottom)
 		)
 	)
